Commit message: Added modified files

File: urdf/udacity_bot.xacro (robot description, xacro)
@@ -184,5 +184,5 @@
       <origin xyz="0 0 0" rpy=" 0 0 0"/>
       <geometry>
-         <mesh filename="package://udacity_bot/meshes/hokuyo.dae"/>
+         <mesh filename="package://slam_project/meshes/hokuyo.dae"/>
       </geometry>
     </visual>

Commit message: Bug fixes

File: urdf/udacity_bot.xacro (robot description, xacro)
@@ -160,4 +160,20 @@
     </visual>
    </link>
+   <link name="camera_rgbd_frame">
+   <inertial>
+     <mass value="0.001" />
+     <origin xyz="0 0 0" />
+     <inertia
+          ixx="1e-6" ixy="0" ixz="0"
+          iyy="1e-6" iyz="0"
+          izz="1e-6"
+     />
+   </inertial>
+  </link>
+  <joint type="fixed" name="camera_rgbd_joint" >
+    <origin xyz="0.001 0 0.001" rpy="0 0 0"/>
+    <child link="camera_rgbd_frame" />
+    <parent link="camera"/>
+  </joint>
    <joint type="fixed" name="camera_joint">
         <origin xyz="0.2 0 0" rpy="0 0 0"/>

Commit message: Inverting laser scan

File: urdf/udacity_bot.xacro (robot description, xacro)
@@ -171,4 +171,14 @@
    </inertial>
   </link>
+ <link name="camera_link_optical">
+ </link>
+ <joint name="camera_optical_joint" type="fixed">
+  <!-- these values have to be these values otherwise the gazebo camera
+      image won't be aligned properly with the frame it is supposedly
+      originating from -->
+  <origin xyz="0 0 0" rpy="${-pi/2} 0 ${-pi/2}"/>
+  <parent link="camera_rgbd_frame"/>
+  <child link="camera_link_optical"/>
+ </joint>
   <joint type="fixed" name="camera_rgbd_joint" >
     <origin xyz="0.001 0 0.001" rpy="0 0 0"/>
@@ -182,5 +192,5 @@
         <axis xyz="0 1 0" rpy="0 0 0"/>
    </joint>
- <link name="hokuyo">
+   <link name="hokuyo">
    <inertial>
       <mass value="0.1"/>
